Commit message: working description

File: manipulator_description/urdf/manipulator.urdf.xacro (robot description, xacro)
@@ -1,18 +1,29 @@
 <?xml version="1.0"?>
 <robot xmlns:xacro="http://ros.org/wiki/xacro" name="ur5_manipulator">
-    <!-- load ur5 robot from ros_industrial/ur_description-->
-    <xacro:include filename="$(find ur_description)/urdf/ur5.xacro" />
-    <!-- include gazbeo ft sensor plugin -->
+    <!-- Define a property to select your robot prefix -->
+    <xacro:property name="robot_prefix" value="ur5_" />
+    <!-- Include base attachment -->
+    <xacro:include filename="$(find manipulator_description)/urdf/base_attachment.urdf.xacro" />
+    <!-- Include UR5 robot from ros_industrial/ur_description -->
+    <xacro:include filename="$(find ur_description)/urdf/inc/ur5_macro.xacro" />
+    <!-- include gripper -->
+    <xacro:include filename="$(find robotiq_gripper)/urdf/robotiq_85_gripper.urdf.xacro" />
+    <!-- Include Gazebo force-torque sensor plugin -->
     <xacro:include filename="$(find manipulator_description)/urdf/ft_sensor.gazebo.xacro" />
+    <!-- Include the file that defines the 'table' macro -->
+    <xacro:include filename="$(find manipulator_description)/urdf/table.urdf.xacro" />
     <!-- Define the world link -->
-    <!-- <link name="world" /> -->
-    <!-- call the ur5 robot -->
-    <xacro:ur5_robot prefix="ur5_"/>
-    <!-- mount plugin to ur5 robot -->
-    <xacro:ft_sensor_gazebo joint="wrist_3_joint"/>
-    <!-- <joint name="ur5_world_fix" type="fixed">
-    <parent link="world" />
-    <child link="base_link" />
-    <origin xyz="0 0 0" rpy="0 0 0" />
-    </joint>     -->
+    <link name="world" />
+    <!-- Call the base attachment using the property value -->
+    <xacro:base_attachment name="${robot_prefix}attachment" parent="world" robot="${robot_prefix}" />
+    <!-- Call the UR5 robot using the property value -->
+    <xacro:ur5_robot prefix="${robot_prefix}"/>
+    <!-- Mount the force-torque sensor plugin to the UR5 robot using the property value -->
+    <xacro:ft_sensor_gazebo joint="${robot_prefix}wrist_3_joint"/>
+    <!-- mount gripper -->
+    <xacro:robotiq_85_gripper prefix="gripper_" parent="${robot_prefix}tool0">
+        <origin xyz="0 0 0" rpy="0 -1.57 0" />
+    </xacro:robotiq_85_gripper>
+    <!-- add table -->
+    <xacro:table name="table" parent="world"/>
 </robot>

Commit message: working gazebo with ur5, no gripper

File: manipulator_description/urdf/manipulator.urdf.xacro (robot description, xacro)
@@ -3,4 +3,5 @@
     <!-- Define a property to select your robot prefix -->
     <xacro:property name="robot_prefix" value="ur5_" />
+    <xacro:property name="transmission_interface" value="hardware_interface/EffortJointInterface" />
     <!-- Include base attachment -->
     <xacro:include filename="$(find manipulator_description)/urdf/base_attachment.urdf.xacro" />
@@ -8,5 +9,5 @@
     <xacro:include filename="$(find ur_description)/urdf/inc/ur5_macro.xacro" />
     <!-- include gripper -->
-    <xacro:include filename="$(find robotiq_gripper)/urdf/robotiq_85_gripper.urdf.xacro" />
+    <!-- <xacro:include filename="$(find robotiq_gripper)/urdf/robotiq_85_gripper.urdf.xacro" /> -->
     <!-- Include Gazebo force-torque sensor plugin -->
     <xacro:include filename="$(find manipulator_description)/urdf/ft_sensor.gazebo.xacro" />
@@ -18,11 +19,11 @@
     <xacro:base_attachment name="${robot_prefix}attachment" parent="world" robot="${robot_prefix}" />
     <!-- Call the UR5 robot using the property value -->
-    <xacro:ur5_robot prefix="${robot_prefix}"/>
+    <xacro:ur5_robot prefix="${robot_prefix}" transmission_hw_interface="${transmission_interface}"/>
     <!-- Mount the force-torque sensor plugin to the UR5 robot using the property value -->
     <xacro:ft_sensor_gazebo joint="${robot_prefix}wrist_3_joint"/>
     <!-- mount gripper -->
-    <xacro:robotiq_85_gripper prefix="gripper_" parent="${robot_prefix}tool0">
+    <!-- <xacro:robotiq_85_gripper prefix="gripper_" parent="${robot_prefix}tool0">
         <origin xyz="0 0 0" rpy="0 -1.57 0" />
-    </xacro:robotiq_85_gripper>
+    </xacro:robotiq_85_gripper> -->
     <!-- add table -->
     <xacro:table name="table" parent="world"/>

File: manipulator_moveit_config/config/gazebo_ur5_manipulator.urdf (robot description, URDF)
Before this commit: robot ur5_manipulator, 27 links, 26 joints
Links:
- removed link gripper_robotiq_85_base_link
- removed link gripper_robotiq_85_left_finger_link
- removed link gripper_robotiq_85_left_finger_tip_link
- removed link gripper_robotiq_85_left_inner_knuckle_link
- removed link gripper_robotiq_85_left_knuckle_link
- removed link gripper_robotiq_85_right_finger_link
- removed link gripper_robotiq_85_right_finger_tip_link
- removed link gripper_robotiq_85_right_inner_knuckle_link
- removed link gripper_robotiq_85_right_knuckle_link
Joints:
- removed joint gripper_robotiq_85_base_joint
- removed joint gripper_robotiq_85_left_finger_joint
- removed joint gripper_robotiq_85_left_finger_tip_joint
- removed joint gripper_robotiq_85_left_inner_knuckle_joint
- removed joint gripper_robotiq_85_left_knuckle_joint
- removed joint gripper_robotiq_85_right_finger_joint
- removed joint gripper_robotiq_85_right_finger_tip_joint
- removed joint gripper_robotiq_85_right_inner_knuckle_joint
- removed joint gripper_robotiq_85_right_knuckle_joint
- joint ur5_base_link-base_fixed_joint: origin xyz=0 0 0 rpy=0 0 3.14159 -> xyz=0 0 0 rpy=0 0 3.141592653589793
- joint ur5_base_link-base_link_inertia: origin xyz=0 0 0 rpy=0 0 3.14159 -> xyz=0 0 0 rpy=0 0 3.141592653589793
- joint ur5_flange-tool0: origin xyz=0 0 0 rpy=1.570795 0 1.570795 -> xyz=0 0 0 rpy=1.5707963267948966 0 1.5707963267948966
- joint ur5_wrist_3-flange: origin xyz=0 0 0 rpy=0 -1.570795 -1.570795 -> xyz=0 0 0 rpy=0 -1.5707963267948966 -1.5707963267948966

Commit message: working gazebo gripper

File: manipulator_description/urdf/manipulator.urdf.xacro (robot description, xacro)
@@ -9,5 +9,5 @@
     <xacro:include filename="$(find ur_description)/urdf/inc/ur5_macro.xacro" />
     <!-- include gripper -->
-    <!-- <xacro:include filename="$(find robotiq_gripper)/urdf/robotiq_85_gripper.urdf.xacro" /> -->
+    <xacro:include filename="$(find robotiq_description)/urdf/robotiq_85_gripper.urdf.xacro" />
     <!-- Include Gazebo force-torque sensor plugin -->
     <xacro:include filename="$(find manipulator_description)/urdf/ft_sensor.gazebo.xacro" />
@@ -23,7 +23,7 @@
     <xacro:ft_sensor_gazebo joint="${robot_prefix}wrist_3_joint"/>
     <!-- mount gripper -->
-    <!-- <xacro:robotiq_85_gripper prefix="gripper_" parent="${robot_prefix}tool0">
+    <xacro:robotiq_85_gripper prefix="gripper_" parent="${robot_prefix}tool0">
         <origin xyz="0 0 0" rpy="0 -1.57 0" />
-    </xacro:robotiq_85_gripper> -->
+    </xacro:robotiq_85_gripper>
     <!-- add table -->
     <xacro:table name="table" parent="world"/>

File: manipulator_description/urdf/manipulator_gripper.urdf (robot description, URDF)
Before this commit: robot ur5_manipulator, 27 links, 26 joints
Links:
- link gripper_robotiq_85_base_link: geometry collision mesh filename=package://robotiq_description/meshes/collision/robotiq_85_b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; visual mesh filename=package://robotiq_description/meshes/visual/robotiq_85_base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
- link gripper_robotiq_85_left_finger_link: geometry collision mesh filename=package://robotiq_description/meshes/collision/robotiq_85_f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; visual mesh filename=package://robotiq_description/meshes/visual/robotiq_85_fing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
- link gripper_robotiq_85_left_finger_tip_link: geometry collision mesh filename=package://robotiq_description/meshes/collision/robotiq_85_f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; visual mesh filename=package://robotiq_description/meshes/visual/robotiq_85_fing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
- link gripper_robotiq_85_left_inner_knuckle_link: geometry collision mesh filename=package://robotiq_description/meshes/collision/robotiq_85_i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; visual mesh filename=package://robotiq_description/meshes/visual/robotiq_85_inne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
- link gripper_robotiq_85_left_knuckle_link: geometry collision mesh filename=package://robotiq_description/meshes/collision/robotiq_85_k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; visual mesh filename=package://robotiq_description/meshes/visual/robotiq_85_knuc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
- link gripper_robotiq_85_right_finger_link: geometry collision mesh filename=package://robotiq_description/meshes/collision/robotiq_85_f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; visual mesh filename=package://robotiq_description/meshes/visual/robotiq_85_fing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
- link gripper_robotiq_85_right_finger_tip_link: geometry collision mesh filename=package://robotiq_description/meshes/collision/robotiq_85_f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; visual mesh filename=package://robotiq_description/meshes/visual/robotiq_85_fing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
- link gripper_robotiq_85_right_inner_knuckle_link: geometry collision mesh filename=package://robotiq_description/meshes/collision/robotiq_85_i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; visual mesh filename=package://robotiq_description/meshes/visual/robotiq_85_inne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
- link gripper_robotiq_85_right_knuckle_link: geometry collision mesh filename=package://robotiq_description/meshes/collision/robotiq_85_k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; visual mesh filename=package://robotiq_description/meshes/visual/robotiq_85_knuc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
Joints:
- removed joint gripper_robotiq_85_left_knuckle_joint
- added joint gripper_finger_joint: type revolute, parent gripper_robotiq_85_base_link, child gripper_robotiq_85_left_knuckle_link, origin xyz=0.05490451627 0.03060114443 0.0 rpy=3.141592653589793 0.0 0.0, axis 0 0 1, limit lower=0.0 upper=0.80285 effort=1000 velocity=0.5
- joint gripper_robotiq_85_left_finger_joint: type continuous -> fixed
- joint gripper_robotiq_85_left_finger_tip_joint: mimic joint=gripper_robotiq_85_left_knuckle_joint multiplier=-1 -> joint=gripper_finger_joint multiplier=-1
- joint gripper_robotiq_85_left_inner_knuckle_joint: mimic joint=gripper_robotiq_85_left_knuckle_joint offset=0 -> joint=gripper_finger_joint offset=0; origin xyz=0.06142 0.0127 0 rpy=3.14159 0.0 0.0 -> xyz=0.06142 0.0127 0 rpy=3.141592653589793 0.0 0.0
- joint gripper_robotiq_85_right_finger_joint: type continuous -> fixed
- joint gripper_robotiq_85_right_finger_tip_joint: mimic joint=gripper_robotiq_85_left_knuckle_joint multiplier=-1 -> joint=gripper_finger_joint multiplier=-1
- joint gripper_robotiq_85_right_inner_knuckle_joint: mimic joint=gripper_robotiq_85_left_knuckle_joint offset=0 -> joint=gripper_finger_joint offset=0
- joint gripper_robotiq_85_right_knuckle_joint: mimic joint=gripper_robotiq_85_left_knuckle_joint -> joint=gripper_finger_joint
- joint ur5_base_link-base_fixed_joint: origin xyz=0 0 0 rpy=0 0 3.14159 -> xyz=0 0 0 rpy=0 0 3.141592653589793
- joint ur5_base_link-base_link_inertia: origin xyz=0 0 0 rpy=0 0 3.14159 -> xyz=0 0 0 rpy=0 0 3.141592653589793
- joint ur5_flange-tool0: origin xyz=0 0 0 rpy=1.570795 0 1.570795 -> xyz=0 0 0 rpy=1.5707963267948966 0 1.5707963267948966
- joint ur5_wrist_3-flange: origin xyz=0 0 0 rpy=0 -1.570795 -1.570795 -> xyz=0 0 0 rpy=0 -1.5707963267948966 -1.5707963267948966

Commit message: working gazbeo simulation

File: manipulator_description/urdf/manipulator.urdf.xacro (robot description, xacro)
@@ -28,3 +28,8 @@
     <!-- add table -->
     <xacro:table name="table" parent="world"/>
+    <!-- Add the gazebo_ros_control plugin to the robot, if out commented dont forget to add in moveit generated urdf -->
+    <!-- <gazebo>
+        <plugin filename="libgazebo_ros_control.so" name="gazebo_ros_control">
+        </plugin>
+    </gazebo> -->
 </robot>

File: manipulator_moveit_config/config/gazebo_ur5_manipulator.urdf (robot description, URDF)
Before this commit: robot ur5_manipulator, 18 links, 17 joints
Links:
- added link gripper_robotiq_85_base_link, mass 0.636951; collision mesh filename=package://robotiq_description/meshes/collision/robotiq_85_b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; visual mesh filename=package://robotiq_description/meshes/visual/robotiq_85_base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
- added link gripper_robotiq_85_left_finger_link, mass 0.027309; collision mesh filename=package://robotiq_description/meshes/collision/robotiq_85_f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; visual mesh filename=package://robotiq_description/meshes/visual/robotiq_85_fing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
- added link gripper_robotiq_85_left_finger_tip_link, mass 0.019555; collision mesh filename=package://robotiq_description/meshes/collision/robotiq_85_f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; visual mesh filename=package://robotiq_description/meshes/visual/robotiq_85_fing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
- added link gripper_robotiq_85_left_inner_knuckle_link, mass 0.029951; collision mesh filename=package://robotiq_description/meshes/collision/robotiq_85_i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; visual mesh filename=package://robotiq_description/meshes/visual/robotiq_85_inne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
- added link gripper_robotiq_85_left_knuckle_link, mass 0.018491; collision mesh filename=package://robotiq_description/meshes/collision/robotiq_85_k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; visual mesh filename=package://robotiq_description/meshes/visual/robotiq_85_knuc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
- added link gripper_robotiq_85_right_finger_link, mass 0.027309; collision mesh filename=package://robotiq_description/meshes/collision/robotiq_85_f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; visual mesh filename=package://robotiq_description/meshes/visual/robotiq_85_fing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
- added link gripper_robotiq_85_right_finger_tip_link, mass 0.019555; collision mesh filename=package://robotiq_description/meshes/collision/robotiq_85_f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; visual mesh filename=package://robotiq_description/meshes/visual/robotiq_85_fing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
- added link gripper_robotiq_85_right_inner_knuckle_link, mass 0.029951; collision mesh filename=package://robotiq_description/meshes/collision/robotiq_85_i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; visual mesh filename=package://robotiq_description/meshes/visual/robotiq_85_inne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
- added link gripper_robotiq_85_right_knuckle_link, mass 0.018491; collision mesh filename=package://robotiq_description/meshes/collision/robotiq_85_k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; visual mesh filename=package://robotiq_description/meshes/visual/robotiq_85_knuc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
Joints:
- added joint gripper_finger_joint: type revolute, parent gripper_robotiq_85_base_link, child gripper_robotiq_85_left_knuckle_link, origin xyz=0.05490451627 0.03060114443 0.0 rpy=3.141592653589793 0.0 0.0, axis 0 0 1, limit lower=0.0 upper=0.80285 effort=1000 velocity=0.5
- added joint gripper_robotiq_85_base_joint: type fixed, parent ur5_tool0, child gripper_robotiq_85_base_link, origin xyz=0 0 0 rpy=0 -1.57 0
- added joint gripper_robotiq_85_left_finger_joint: type fixed, parent gripper_robotiq_85_left_knuckle_link, child gripper_robotiq_85_left_finger_link, origin xyz=-0.00408552455 -0.03148604435 0.0 rpy=0 0 0
- added joint gripper_robotiq_85_left_finger_tip_joint: type continuous, parent gripper_robotiq_85_left_inner_knuckle_link, child gripper_robotiq_85_left_finger_tip_link, origin xyz=0.04303959807 -0.03759940821 0.0 rpy=0.0 0.0 0.0, axis 0 0 1, limit lower=-3.14 upper=3.14 effort=0.1 velocity=100.0, mimic joint=gripper_finger_joint multiplier=-1
- added joint gripper_robotiq_85_left_inner_knuckle_joint: type continuous, parent gripper_robotiq_85_base_link, child gripper_robotiq_85_left_inner_knuckle_link, origin xyz=0.06142 0.0127 0 rpy=3.141592653589793 0.0 0.0, axis 0 0 1, limit lower=-3.14 upper=3.14 effort=0.1 velocity=100.0, mimic joint=gripper_finger_joint offset=0
- added joint gripper_robotiq_85_right_finger_joint: type fixed, parent gripper_robotiq_85_right_knuckle_link, child gripper_robotiq_85_right_finger_link, origin xyz=-0.00408552455 -0.03148604435 0.0 rpy=0 0 0
- added joint gripper_robotiq_85_right_finger_tip_joint: type continuous, parent gripper_robotiq_85_right_inner_knuckle_link, child gripper_robotiq_85_right_finger_tip_link, origin xyz=0.04303959807 -0.03759940821  0.0 rpy=0.0 0.0 0.0, axis 0 0 1, limit lower=-3.14 upper=3.14 effort=0.1 velocity=100.0, mimic joint=gripper_finger_joint multiplier=-1
- added joint gripper_robotiq_85_right_inner_knuckle_joint: type continuous, parent gripper_robotiq_85_base_link, child gripper_robotiq_85_right_inner_knuckle_link, origin xyz=0.06142 -0.0127 0 rpy=0 0 0, axis 0 0 1, limit lower=-3.14 upper=3.14 effort=0.1 velocity=100.0, mimic joint=gripper_finger_joint offset=0
- added joint gripper_robotiq_85_right_knuckle_joint: type continuous, parent gripper_robotiq_85_base_link, child gripper_robotiq_85_right_knuckle_link, origin xyz=0.05490451627 -0.03060114443 0.0 rpy=0.0 0.0 0.0, axis 0 0 1, limit lower=-3.14 upper=3.14 effort=1000 velocity=100.0, mimic joint=gripper_finger_joint

Commit message: added ft_sensor mesh

File: manipulator_description/urdf/manipulator.urdf.xacro (robot description, xacro)
@@ -4,12 +4,16 @@
     <xacro:property name="robot_prefix" value="ur5_" />
     <xacro:property name="transmission_interface" value="hardware_interface/EffortJointInterface" />
+    <xacro:property name="ft_prefix" value="sensor_" />
+    <xacro:property name="gripper_prefix" value="gripper_" />
     <!-- Include base attachment -->
     <xacro:include filename="$(find manipulator_description)/urdf/base_attachment.urdf.xacro" />
     <!-- Include UR5 robot from ros_industrial/ur_description -->
     <xacro:include filename="$(find ur_description)/urdf/inc/ur5_macro.xacro" />
+    <!-- include force-torque sensor -->
+    <xacro:include filename="$(find robotiq_ft_sensor)/urdf/robotiq_ft300.urdf.xacro" />
+    <!-- Include Gazebo force-torque sensor plugin -->
+    <xacro:include filename="$(find manipulator_description)/urdf/ft_sensor.gazebo.xacro" />
     <!-- include gripper -->
     <xacro:include filename="$(find robotiq_description)/urdf/robotiq_85_gripper.urdf.xacro" />
-    <!-- Include Gazebo force-torque sensor plugin -->
-    <xacro:include filename="$(find manipulator_description)/urdf/ft_sensor.gazebo.xacro" />
     <!-- Include the file that defines the 'table' macro -->
     <xacro:include filename="$(find manipulator_description)/urdf/table.urdf.xacro" />
@@ -20,8 +24,11 @@
     <!-- Call the UR5 robot using the property value -->
     <xacro:ur5_robot prefix="${robot_prefix}" transmission_hw_interface="${transmission_interface}"/>
-    <!-- Mount the force-torque sensor plugin to the UR5 robot using the property value -->
-    <xacro:ft_sensor_gazebo joint="${robot_prefix}wrist_3_joint"/>
+    <!-- Mount the force-torque sensor & plugin to the UR5 -->
+     <xacro:robotiq_ft300 parent="${robot_prefix}tool0" prefix="${ft_prefix}">
+        <origin xyz="0 0 -0.004" rpy="0 0 0"/>
+    </xacro:robotiq_ft300>
+    <xacro:ft_sensor_gazebo joint="${ft_prefix}measurment_joint"/>
     <!-- mount gripper -->
-    <xacro:robotiq_85_gripper prefix="gripper_" parent="${robot_prefix}tool0">
+    <xacro:robotiq_85_gripper prefix="${gripper_prefix}" parent="${ft_prefix}robotiq_ft_frame_id">
         <origin xyz="0 0 0" rpy="0 -1.57 0" />
     </xacro:robotiq_85_gripper>
@@ -29,7 +36,7 @@
     <xacro:table name="table" parent="world"/>
     <!-- Add the gazebo_ros_control plugin to the robot, if out commented dont forget to add in moveit generated urdf -->
-    <!-- <gazebo>
+    <gazebo>
         <plugin filename="libgazebo_ros_control.so" name="gazebo_ros_control">
         </plugin>
-    </gazebo> -->
+    </gazebo>
 </robot>

File: manipulator_moveit_config/config/gazebo_ur5_manipulator.urdf (robot description, URDF)
Before this commit: robot ur5_manipulator, 27 links, 26 joints
Links:
- added link sensor_ft300_mounting_plate, mass 0.1; collision mesh filename=package://robotiq_ft_sensor/meshes/collision/mountings/robo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; visual mesh filename=package://robotiq_ft_sensor/meshes/visual/mountings/robotiq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
- added link sensor_ft300_sensor, mass 0.300; collision mesh filename=package://robotiq_ft_sensor/meshes/collision/robotiq_ft300.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; visual mesh filename=package://robotiq_ft_sensor/meshes/visual/robotiq_ft300.STL
- added link sensor_robotiq_ft_frame_id
Joints:
- added joint sensor_ft300_fix: type fixed, parent ur5_tool0, child sensor_ft300_mounting_plate, origin xyz=0 0 -0.004 rpy=0 0 0
- added joint sensor_ft300_mounting_plate: type fixed, parent sensor_ft300_mounting_plate, child sensor_ft300_sensor, origin xyz=0 0 0.0415 rpy=0 3.141592653589793 0
- added joint sensor_measurment_joint: type revolute, parent sensor_ft300_sensor, child sensor_robotiq_ft_frame_id, origin xyz=0 0 0 rpy=0 3.141592653589793 -1.5707963267948966, limit lower=0 upper=0 effort=0 velocity=0
- joint gripper_robotiq_85_base_joint: parent ur5_tool0 -> sensor_robotiq_ft_frame_id
