Commit message: corrected moveit_config positions & collision

File: manipulator_description/urdf/base_attachment.urdf.xacro (robot description, xacro)
@@ -7,5 +7,5 @@
         <parent link="${parent}"/>
         <child link="${name}_base_link"/>
-        <origin xyz="0 0.6 0.425" rpy="0 0 -1.5708"/> <!-- Lift by half the cylinder height -->
+        <origin xyz="-0.095725 0.65 0.425" rpy="0 0 -1.5708"/> <!-- Lift by half the cylinder height -->
     </joint>
     <!-- Grey Cylinder Base -->

File: manipulator_description/urdf/manipulator.urdf.xacro (robot description, xacro)
@@ -17,5 +17,5 @@
     <xacro:include filename="$(find robotiq_description)/urdf/robotiq_85_gripper.urdf.xacro" />
     <!-- Include the file that defines the 'table' macro -->
-    <xacro:include filename="$(find manipulator_description)/urdf/table.urdf.xacro" />
+    <xacro:include filename="$(find manipulator_description)/urdf/table/table.urdf.xacro" />
     <!-- Define the world link -->
     <link name="world" />

File: manipulator_moveit_config/config/gazebo_ur5_manipulator.urdf (robot description, URDF)
Before this commit: robot ur5_manipulator, 30 links, 29 joints
Links:
- removed link table_back_left_leg
- removed link table_back_right_leg
- removed link table_front_left_leg
- removed link table_front_right_leg
- removed link table_top_link
- added link table_baseLink, mass 1.0; collision box size=1.5 1 0.05; visual mesh filename=package://manipulator_description/urdf/table/table.obj scale=0.1 0.1 0.58
Joints:
- removed joint table_back_left_leg_joint
- removed joint table_back_right_leg_joint
- removed joint table_front_left_leg_joint
- removed joint table_front_right_leg_joint
- removed joint table_to_parent
- added joint table_to_world: type fixed, parent world, child table_baseLink, origin xyz=0 0 0 rpy=0 0 0
- joint ur5_attachment_to_world: origin xyz=0 0.6 0.425 rpy=0 0 -1.5708 -> xyz=-0.095725 0.65 0.425 rpy=0 0 -1.5708

Commit message: updated collision attachment, logs in preprocess

File: manipulator_description/urdf/base_attachment.urdf.xacro (robot description, xacro)
@@ -22,5 +22,5 @@
       <collision>
         <geometry>
-          <cylinder radius="0.3" length="0.5"/>
+          <cylinder radius="0.1" length="0.85"/>
         </geometry>
         <origin xyz="0 0 0" rpy="0 0 0"/>

File: manipulator_moveit_config/config/gazebo_ur5_manipulator.urdf (robot description, URDF)
Before this commit: robot ur5_manipulator, 26 links, 25 joints
Links:
- link ur5_attachment_base_link: geometry collision cylinder length=0.85 radius=0.1; visual cylinder length=0.85 radius=0.1
